Commit message: Update d435.xacro

File: legged_rl-go1_student_deploy/legged_robot/legged_unitree/legged_unitree_description/urdf/common/d435.xacro (robot description, xacro)
@@ -7,5 +7,5 @@
         <joint name="camera_depth_joint" type="fixed">
             <!-- 相机连接的位置 -->
-            <origin xyz="0.27 0.015 0.086" rpy="0 0.0 0"/>
+            <origin xyz="0.27 0.015 0.086" rpy="0 1.2 0"/>
             <!-- 父链接 -->
             <parent link="${connected_to}"/>
